File: Hardware/Scicalc.kicad_sch (KiCad schematic)
At the start: 138 parts, among them J1 USB_C_Receptacle_USB2.0_16P, J2 Conn_01x02_Pin, J3 Conn_01x09_Pin, SW1 SW_Push, SW10 SW_Push, SW11 SW_Push, SW12 SW_Push, SW13 SW_Push, SW14 SW_Push, SW15 SW_Push, SW16 SW_Push, SW17 SW_Push, SW18 SW_Push, SW19 SW_Push, SW2 SW_Push, SW20 SW_Push, SW21 SW_Push, SW22 SW_Push, SW23 SW_Push, SW24 SW_Push, SW25 SW_Push, SW26 SW_Push, SW27 SW_Push, SW28 SW_Push, SW29 SW_Push, SW3 SW_Push, SW30 SW_Push, SW31 SW_Push, SW32 SW_Push, SW33 SW_Push, SW34 SW_Push, SW35 SW_Push, SW36 SW_Push, SW37 SW_Push, SW38 SW_Push, SW39 SW_Push, SW4 SW_Push, SW40 SW_Push, SW41 SW_Push, SW42 SW_Push, SW43 SW_Push, SW44 SW_Push, SW45 SW_Push, SW46 SW_Push, SW47 SW_Push, SW48 SW_Push, SW49 SW_Push, SW5 SW_Push, SW50 SW_Push, SW51 SW_Push, SW6 SW_Push, SW7 SW_Push, SW8 SW_Push, SW9 SW_Push, U1 RP2350A, U2 MCP1700x-330xxTT, U3 W25Q128JVP, U5 RM2, U6 BQ24075RGT, Y1 12 mhz

Commit message: Completed PCB
Connections:
- net OUT is gone; now on net VBUS: C18.1, U6.10 (OUT), U6.11 (OUT)
- net COL-1: now also U1.8 (GPIO5); no longer U1.18 (GPIO14)
- net COL-10: now also U1.18 (GPIO14); no longer U1.8 (GPIO5)
- net COL-2: now also U1.9 (GPIO6); no longer U1.17 (GPIO13)
- net COL-3: now also U1.10 (GPIO7); no longer U1.16 (GPIO12)
- net COL-4: now also U1.12 (GPIO8); no longer U1.15 (GPIO11)
- net COL-5: now also U1.13 (GPIO9); no longer U1.14 (GPIO10)
- net COL-6: now also U1.14 (GPIO10); no longer U1.13 (GPIO9)
- net COL-7: now also U1.15 (GPIO11); no longer U1.12 (GPIO8)
- net COL-8: now also U1.16 (GPIO12); no longer U1.10 (GPIO7)
- net COL-9: now also U1.17 (GPIO13); no longer U1.9 (GPIO6)
- net GND: now also R3.2, R4.2
- net GP25: now also U1.37 (GPIO25)
- net ROW-1: now also U1.7 (GPIO4); no longer U1.2 (GPIO0)
- net ROW-2: now also U1.5 (GPIO3); no longer U1.3 (GPIO1)
- net ROW-4: now also U1.3 (GPIO1); no longer U1.5 (GPIO3)
- net ROW-5: now also U1.2 (GPIO0); no longer U1.7 (GPIO4)
- no-connect marks 14 -> 12
Changed lines of the file:
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@@
 	)
 	(junction
+		(at 107.95 308.61)
+		(diameter 0)
+		(color 0 0 0 0)
+	)
+	(junction
 		(at 495.3 85.09)
 		(diameter 0)
@@
 	)
 	(no_connect
-		(at 231.14 170.18)
-	)
-	(no_connect
 		(at 231.14 177.8)
 	)
@@
 	)
 	(no_connect
-		(at 231.14 175.26)
-	)
-	(no_connect
 		(at 231.14 160.02)
 	)
@@
 	(wire
 		(pts
+			(xy 107.95 308.61) (xy 115.57 308.61)
+		)
+		(stroke
+			(width 0)
+			(type default)
+		)
+	)
+	(wire
+		(pts
 			(xy 505.46 130.81) (xy 488.95 130.81)
 		)
@@
 	(wire
 		(pts
+			(xy 107.95 308.61) (xy 107.95 323.85)
+		)
+		(stroke
+			(width 0)
+			(type default)
+		)
+	)
+	(wire
+		(pts
 			(xy 44.45 246.38) (xy 45.72 246.38)
 		)
@@
 	(wire
 		(pts
-			(xy 95.25 308.61) (xy 115.57 308.61)
+			(xy 95.25 308.61) (xy 107.95 308.61)
 		)
 		(stroke
@@
 		)
 	)
-	(label "COL-2"
-		(at 231.14 139.7 0)
+	(label "ROW-1"
+		(at 231.14 116.84 0)
 		(effects
 			(font
@@
 		)
 	)
-	(label "COL-10"
-		(at 231.14 119.38 0)
-		(effects
-			(font
-				(size 1.27 1.27)
-			)
-			(justify left bottom)
-		)
-	)
 	(label "QSPI_CLK"
 		(at 180.34 142.24 180)
@@
 		)
 	)
-	(label "COL-3"
-		(at 231.14 137.16 0)
-		(effects
-			(font
-				(size 1.27 1.27)
-			)
-			(justify left bottom)
-		)
-	)
 	(label "BAT+"
 		(at 107.95 331.47 0)
@@
 		)
 	)
-	(label "COL-4"
-		(at 231.14 134.62 0)
-		(effects
-			(font
-				(size 1.27 1.27)
-			)
-			(justify left bottom)
-		)
-	)
 	(label "USB_D-"
 		(at 71.12 123.19 180)
@@
 		)
 	)
-	(label "GP24"
-		(at 267.97 332.74 0)
+	(label "COL-9"
+		(at 231.14 139.7 0)
 		(effects
 			(font
@@
 		)
 	)
-	(label "COL-7"
-		(at 231.14 127 0)
+	(label "GP24"
+		(at 267.97 332.74 0)
 		(effects
 			(font
@@
 		)
 	)
-	(label "ROW-5"
-		(at 231.14 116.84 0)
+	(label "GP23"
+		(at 231.14 165.1 0)
 		(effects
 			(font
@@
 		)
 	)
-	(label "GP23"
-		(at 231.14 165.1 0)
+	(label "ROW-5"
+		(at 231.14 106.68 0)
 		(effects
 			(font
@@
 		)
 	)
-	(label "COL-5"
-		(at 231.14 132.08 0)
+	(label "RUN"
+		(at 180.34 121.92 180)
 		(effects
 			(font
 				(size 1.27 1.27)
 			)
-			(justify left bottom)
+			(justify right bottom)
 		)
 	)
-	(label "RUN"
-		(at 180.34 121.92 180)
+	(label "COL-7"
+		(at 231.14 134.62 0)
 		(effects
 			(font
 				(size 1.27 1.27)
 			)
-			(justify right bottom)
+			(justify left bottom)
 		)
 	)
@@
 	)
 	(label "COL-9"
-		(at 231.14 121.92 0)
+		(at 443.23 226.06 0)
 		(effects
 			(font
@@
 	)
 	(label "ROW-4"
-		(at 231.14 114.3 0)
+		(at 231.14 109.22 0)
 		(effects
 			(font
@@
 		)
 	)
-	(label "COL-8"
-		(at 231.14 124.46 0)
+	(label "COL-4"
+		(at 231.14 127 0)
 		(effects
 			(font
@@
 		)
 	)
-	(label "COL-9"
-		(at 443.23 226.06 0)
+	(label "USB_D-"
+		(at 172.72 129.54 180)
 		(effects
 			(font
 				(size 1.27 1.27)
 			)
-			(justify left bottom)
+			(justify right bottom)
 		)
 	)
-	(label "USB_D-"
-		(at 172.72 129.54 180)
+	(label "COL-6"
+		(at 231.14 132.08 0)
 		(effects
 			(font
 				(size 1.27 1.27)
 			)
-			(justify right bottom)
+			(justify left bottom)
 		)
 	)
@@
 		)
 	)
-	(label "GP24"
-		(at 231.14 167.64 0)
+	(label "ROW-3"
+		(at 231.14 111.76 0)
 		(effects
 			(font
@@
 		)
 	)
-	(label "ROW-3"
-		(at 231.14 111.76 0)
+	(label "GP24"
+		(at 231.14 167.64 0)
 		(effects
 			(font
@@
 		)
 	)
-	(label "ROW-1"
-		(at 231.14 106.68 0)
-		(effects
-			(font
-				(size 1.27 1.27)
-			)
-			(justify left bottom)
-		)
-	)
 	(label "USB_D+"
 		(at 71.12 128.27 180)
@@
 		)
 	)
-	(label "ROW-2"
-		(at 231.14 109.22 0)
-		(effects
-			(font
-				(size 1.27 1.27)
-			)
-			(justify left bottom)
-		)
-	)
 	(label "EN"
 		(at 231.14 144.78 0)
@@
 		)
 	)
+	(label "COL-8"
+		(at 231.14 137.16 0)
+		(effects
+			(font
+				(size 1.27 1.27)
+			)
+			(justify left bottom)
+		)
+	)
+	(label "COL-1"
+		(at 231.14 119.38 0)
+		(effects
+			(font
+				(size 1.27 1.27)
+			)
+			(justify left bottom)
+		)
+	)
 	(label "QSPI_CLK"
 		(at 59.69 186.69 0)
@@
 		)
 	)
+	(label "GP25"
+		(at 231.14 170.18 0)
+		(effects
+			(font
+				(size 1.27 1.27)
+			)
+			(justify left bottom)
+		)
+	)
 	(label "CHG"
 		(at 107.95 344.17 0)
@@
 		)
 	)
-	(label "COL-6"
-		(at 231.14 129.54 0)
+	(label "COL-10"
+		(at 231.14 142.24 0)
 		(effects
 			(font
@@
 		)
 	)
+	(label "COL-3"
+		(at 231.14 124.46 0)
+		(effects
+			(font
+				(size 1.27 1.27)
+			)
+			(justify left bottom)
+		)
+	)
+	(label "COL-2"
+		(at 231.14 121.92 0)
+		(effects
+			(font
+				(size 1.27 1.27)
+			)
+			(justify left bottom)
+		)
+	)
 	(label "COL-4"
 		(at 443.23 130.81 0)
@@
 		)
 	)
-	(label "COL-1"
-		(at 231.14 142.24 0)
-		(effects
-			(font
-				(size 1.27 1.27)
-			)
-			(justify left bottom)
-		)
-	)
 	(label "SDA"
 		(at 356.87 326.39 0)
@@
 		)
 	)
+	(label "ROW-2"
+		(at 231.14 114.3 0)
+		(effects
+			(font
+				(size 1.27 1.27)
+			)
+			(justify left bottom)
+		)
+	)
 	(label "XIN"
 		(at 180.34 160.02 180)
@@
 		)
 	)
+	(label "COL-5"
+		(at 231.14 129.54 0)
+		(effects
+			(font
+				(size 1.27 1.27)
+			)
+			(justify left bottom)
+		)
+	)
 	(label "QSPI_IO2"
 		(at 180.34 149.86 180)
@@
 	(symbol
 		(lib_id "power:GND")
-		(at 78.74 120.65 0)
+		(at 78.74 119.38 0)
 		(unit 1)
 		(body_style 1)
@@
 		(fields_autoplaced yes)
 		(property "Reference" "#PWR01"
-			(at 78.74 127 0)
+			(at 78.74 125.73 0)
 			(hide yes)
 			(show_name no)
@@
 		)
 		(property "Value" "GND"
-			(at 78.74 125.73 0)
+			(at 78.74 124.46 0)
 			(show_name no)
 			(do_not_autoplace no)
@@
 		)
 		(property "Footprint" ""
-			(at 78.74 120.65 0)
+			(at 78.74 119.38 0)
 			(hide yes)
 			(show_name no)
@@
 		)
 		(property "Datasheet" ""
-			(at 78.74 120.65 0)
+			(at 78.74 119.38 0)
 			(hide yes)
 			(show_name no)
@@
 		)
 		(property "Description" "Power symbol creates a global label with name \"GND\" , ground"
-			(at 78.74 120.65 0)
+			(at 78.74 119.38 0)
 			(hide yes)
 			(show_name no)
