File: Hardware/Scicalc.kicad_pcb (KiCad board)
At the start: 2 copper layers, 50 x 70 mm, 138 parts, among them J1 USB_C_Receptacle_USB2.0_16P, J2 Conn_01x02_Pin, J3 Conn_01x09_Pin, SW1 SW_Push, SW10 SW_Push, SW11 SW_Push, SW12 SW_Push, SW13 SW_Push, SW14 SW_Push, SW15 SW_Push, SW16 SW_Push, SW17 SW_Push, SW18 SW_Push, SW19 SW_Push, SW2 SW_Push, SW20 SW_Push, SW21 SW_Push, SW22 SW_Push, SW23 SW_Push, SW24 SW_Push, SW25 SW_Push, SW26 SW_Push, SW27 SW_Push, SW28 SW_Push, SW29 SW_Push, SW3 SW_Push, SW30 SW_Push, SW31 SW_Push, SW32 SW_Push, SW33 SW_Push, SW34 SW_Push, SW35 SW_Push, SW36 SW_Push, SW37 SW_Push, SW38 SW_Push, SW39 SW_Push, SW4 SW_Push, SW40 SW_Push, SW41 SW_Push, SW42 SW_Push, SW43 SW_Push, SW44 SW_Push, SW45 SW_Push, SW46 SW_Push, SW47 SW_Push, SW48 SW_Push, SW49 SW_Push, SW5 SW_Push, SW50 SW_Push, SW51 SW_Push, SW6 SW_Push, SW7 SW_Push, SW8 SW_Push, SW9 SW_Push, U1 RP2350A, U2 MCP1700x-330xxTT, U3 W25Q128JVP, U5 RM2, U6 BQ24075RGT, Y1 12 mhz

Commit message: Completed PCB
Parts:
- L1: footprint Inductor_SMD:L_0805_2012Metric -> Inductor_SMD:L_0603_1608Metric
- moved J2 224.6 mm to (133.2, 37.4)
- moved D53 223.7 mm to (135.9, 43.1), turned to -90 degrees
- moved D54 223.0 mm to (136.9, 43.1), turned to -90 degrees
- moved R10 220.5 mm to (140.4, 37.1)
- moved U6 220.5 mm to (138.3, 39.7), turned to -90 degrees
- moved R11 220.1 mm to (141.0, 38.1)
- moved C17 207.0 mm to (135.8, 37.0), turned to 90 degrees
- moved C18 202.0 mm to (140.3, 41.9)
- moved C19 201.5 mm to (141.3, 40.4)
- moved U2 187.9 mm to (171.3, 38.6)
- moved R8 186.6 mm to (171.0, 91.5), turned to 90 degrees
- moved R9 184.7 mm to (175.5, 84.6), turned to 90 degrees
- moved R4 183.4 mm to (174.4, 39.3), turned to 180 degrees
- moved SW1 181.7 mm to (181.0, 82.2), turned to 90 degrees
- moved R3 180.6 mm to (174.4, 42.3), turned to 180 degrees
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Connections:
- C18 pad 1: /OUT -> VBUS
- R3 pad 2: Net-(R3-Pad2) -> GND
- R4 pad 2: Net-(R3-Pad2) -> GND
- U1 pad 10: /COL-8 -> /COL-3
- U1 pad 12: /COL-7 -> /COL-4
- U1 pad 13: /COL-6 -> /COL-5
- U1 pad 14: /COL-5 -> /COL-6
- U1 pad 15: /COL-4 -> /COL-7
- U1 pad 16: /COL-3 -> /COL-8
- U1 pad 17: /COL-2 -> /COL-9
- U1 pad 18: /COL-1 -> /COL-10
- U1 pad 2: /ROW-1 -> /ROW-5
- U1 pad 3: /ROW-2 -> /ROW-4
- U1 pad 37: unconnected-(U1-GPIO25-Pad37) -> /GP25
- U1 pad 5: /ROW-4 -> /ROW-2
- U1 pad 7: /ROW-5 -> /ROW-1
- U1 pad 8: /COL-10 -> /COL-1
- U1 pad 9: /COL-9 -> /COL-2
- U6 pad 10: /OUT -> VBUS
- U6 pad 11: /OUT -> VBUS
Routing:
- net /ROW-1: track 0.00 -> 92.6 mm, vias 0 -> 2
- net /ROW-2: track 0.00 -> 85.5 mm, vias 0 -> 2
- net /ROW-3: track 0.00 -> 78.6 mm, vias 0 -> 2
- net /ROW-4: track 0.00 -> 76.0 mm, vias 0 -> 2
- net /COL-10: track 0.00 -> 71.5 mm, vias 0 -> 2
- net /COL-1: track 0.00 -> 67.9 mm, vias 0 -> 6
- net /ROW-5: track 0.00 -> 65.6 mm, vias 0 -> 2
- net /COL-9: track 0.00 -> 61.6 mm, vias 0 -> 6
- net /COL-2: track 0.00 -> 56.6 mm, vias 0 -> 6
- net /SCL: track 0.00 -> 56.4 mm, vias 0 -> 1
- net /COL-3: track 0.00 -> 55.2 mm, vias 0 -> 5
- net /COL-8: track 0.00 -> 54.6 mm, vias 0 -> 6
- net +3V3: track 6.05 -> 59.6 mm, vias 0 -> 17
- net /EN: track 0.00 -> 52.4 mm, vias 0 -> 2
- net /CS: track 0.00 -> 50.8 mm, vias 0 -> 1
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- added copper zone on In2.Cu, net +3V3
- added copper zone on B.Cu, net GND
- added copper zone on F.Cu, net GND
- added copper zone on In1.Cu, net GND
Other:
- board size 50 x 70 mm -> 52.9 x 70 mm
- copper layers 2 -> 4

Commit message: added latest images, updated readme, gitignore
Parts:
- added REF**: MountingHole_3.2mm_M3, MountingHole:MountingHole_3.2mm_M3, B.Cu at (170.8, 82.6)
- added REF**: MountingHole_3.2mm_M3, MountingHole:MountingHole_3.2mm_M3, B.Cu at (145.1, 42.7)
- added REF**: MountingHole_3.2mm_M3, MountingHole:MountingHole_3.2mm_M3, B.Cu at (177.2, 58.4)
Routing:
- net /COL-8: track 54.6 -> 56.3 mm
